File: PCB/PCB.kicad_sch (KiCad schematic)
At the start: 0 parts

Commit message: adding in the artix FPGA symbol
Parts:
- added U1, U2: XC7A50T-FGG484, symbol FPGA_Xilinx_Artix7:XC7A50T-FGG484

Commit message: added in the FPGA footpritn
Parts:
- U1: footprint (none) -> Package_BGA:Xilinx_FGG484
- U1: renamed from U2; footprint (none) -> Package_BGA:Xilinx_FGG484
Changed lines of the file:
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@@
 			)
 		)
-		(property "Footprint" ""
+		(property "Footprint" "Package_BGA:Xilinx_FGG484"
 			(at 355.6 229.87 0)
 			(effects
@@
 			)
 		)
-		(property "Footprint" ""
+		(property "Footprint" "Package_BGA:Xilinx_FGG484"
 			(at 242.57 231.14 0)
 			(effects
@@
 		(dnp no)
 		(fields_autoplaced yes)
-		(property "Reference" "U2"
+		(property "Reference" "U1"
 			(at 91.44 118.7449 0)
 			(effects
@@
 			)
 		)
-		(property "Footprint" ""
+		(property "Footprint" "Package_BGA:Xilinx_FGG484"
 			(at 137.16 116.84 0)
 			(effects
@@
 			(project ""
 				(path "/ed0095eb-57a0-4856-9ac4-7b40bd214a3a"
-					(reference "U2")
+					(reference "U1")
 					(unit 1)
 				)
@@
 			)
 		)
-		(property "Footprint" ""
+		(property "Footprint" "Package_BGA:Xilinx_FGG484"
 			(at 48.26 201.93 0)
 			(effects
@@
 			)
 		)
-		(property "Footprint" ""
+		(property "Footprint" "Package_BGA:Xilinx_FGG484"
 			(at 138.43 234.95 0)
 			(effects
@@
 			)
 		)
-		(property "Footprint" ""
+		(property "Footprint" "Package_BGA:Xilinx_FGG484"
 			(at 361.95 115.57 0)
 			(effects
@@
 			)
 		)
-		(property "Footprint" ""
+		(property "Footprint" "Package_BGA:Xilinx_FGG484"
 			(at 250.19 114.3 0)
 			(effects
