File: PCB/FPGA-power.kicad_sch (KiCad schematic)
At the start: 2 parts, among them U1 XC7A50T-FGG484

Commit message: properly wired the analog and battery pins, did VCCINT decoupling
Parts:
- added C16, C17, C18, C19, C20: 470nF, symbol Device:C
- added C21, C22, C23: 4.7uF, symbol Device:C
- added C24: 330uF, symbol Device:C
Connections:
- net +1V0: now also U1.J11 (VCCBRAM), U1.L11 (VCCBRAM), U1.N11 (VCCBRAM), C16.1, C17.1, C18.1, C19.1, C20.1, C21.1, C22.1, C23.1, C24.1
- net +1V8: no longer U1.E12 (VCCBATT_0), U1.J11 (VCCBRAM), U1.K9 (GNDADC_0), U1.L11 (VCCBRAM), U1.N11 (VCCBRAM)
- net GND: now also U1.E12 (VCCBATT_0), U1.K9 (GNDADC_0), C16.2, C17.2, C18.2, C19.2, C20.2, C21.2, C22.2, C23.2, C24.2
Other:
- moved on the sheet: R1, U1E

Commit message: VCCBRAM decoupling!
Parts:
- added C25: 470nF, symbol Device:C
- added C26: 100uF, symbol Device:C
Connections:
- net +1V0: now also C25.1, C26.1
- net GND: now also C25.2, C26.2
