File: PCB/FPGA-power.kicad_sch (KiCad schematic)
At the start: 24 parts, among them U1 XC7A50T-FGG484

Commit message: finished decoupling, cleaned it up, and journaled about it
Parts:
- added C38, C39: 470nF, symbol Device:C
- added C40: 4.7uF, symbol Device:C
Connections:
- net +1V2: now also C38.1, C39.1, C40.1
- net GND: now also C38.2, C39.2, C40.2
Other:
- moved on the sheet: C16, C17, C18, C19, C20, C21, C22, C23, C24, C25, C26, C27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
