File: PCB/FPGA-power.kicad_sch (KiCad schematic)
At the start: 33 parts, among them U1 XC7A50T-FGG484

Commit message: journaling  about the ferrite beads
Other:
- note removed: "FERRITE BEADS AND ANALOG RAILS"
Changed lines of the file:
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@@
-		)
-	)
-	(text "FERRITE BEADS AND ANALOG RAILS"
-		(exclude_from_sim no)
-		(at 58.42 -1.524 0)
-		(effects
-			(font
-				(size 3.81 3.81)
-			)
 		)
 	)
