File: PCB/power.kicad_sch (KiCad schematic)
At the start: 23 parts, among them U2 LTC3370

Commit message: fixed schematic, journaled about quad buck
Parts:
- L1, L2, L3, L4: value 22u -> 2.2u
Changed lines of the file:
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@@
 			)
 		)
-		(property "Value" "22u"
+		(property "Value" "2.2u"
 			(at 175.26 74.676 90)
 			(effects
@@
 			)
 		)
-		(property "Value" "22u"
+		(property "Value" "2.2u"
 			(at 109.22 103.886 90)
 			(effects
@@
 			)
 		)
-		(property "Value" "22u"
+		(property "Value" "2.2u"
 			(at 175.26 103.886 90)
 			(effects
@@
 			)
 		)
-		(property "Value" "22u"
+		(property "Value" "2.2u"
 			(at 109.22 74.676 90)
 			(effects
