File: PCB/power.kicad_sch (KiCad schematic)
At the start: 27 parts, among them U2 MAX20029ATIA/V+

Commit message: created the TPS2121 symbol
Parts:
- added U5: TPS2121RUXR, Package_DFN_QFN:Texas_VQFN-HR-12_2x2.5mm_P0.5mm_ThermalVias, symbol FPGA Accelerator:TPS2121RUXR
Connections:
- new net OUT: U5.1 (OUT), U5.8 (OUT)
Other:
- moved on the sheet: C41, C42, C43, C44, C45, C46, C48, C49, C50, C51, C52, C53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
