File: PCB/configurations.kicad_sch (KiCad schematic)
At the start: 5 parts, among them U1 XC7A50T-FGG484

Commit message: wired a basic JTAG TC2030
Parts:
- added J2: Conn_ARM_SWD_TagConnect_TC2030, Connector:Tag-Connect_TC2030-IDC-FP_2x03_P1.27mm_Vertical, symbol Connector:Conn_ARM_SWD_TagConnect_TC2030
- added J3: USB_C_Receptacle_USB2.0_16P, Connector_USB:USB_C_Receptacle_HRO_TYPE-C-31-M-12, symbol Connector:USB_C_Receptacle_USB2.0_16P
- added R16, R17, R18, R19: 22, symbol Device:R
- added R20, R21: 5.1K, symbol Device:R
- added R22, R23: 10k, symbol Device:R
Connections:
- net +3V3: now also J2.1 (VCC), R22.1, R23.1
- net GND: now also J2.5 (GND), J3.A1 (GND), J3.A12 (GND), J3.B1 (GND), J3.B12 (GND), J3.S1 (SHIELD), R20.2, R21.2
- net TDI: now reaches U1.R13 (TDI_0)
- net TDI: now also R19.2
- net TMS: now reaches U1.T13 (TMS_0)
- net TMS: now also R17.2, R23.2
- net TDO: now reaches U1.U13 (TDO_0)
- net TDO: now also R18.2
- net TCK: now reaches U1.V12 (TCK_0)
- net TCK: now also R16.2, R22.2
- new net: J2.2 (SWDIO), R17.1
- new net: J3.B5 (CC2), R21.1
- new net: J2.6 (SWO), R18.1
- new net: J2.4 (SWCLK), R16.1
- new net: J2.3 (~{RESET}), R19.1
- new net: J3.A4 (VBUS), J3.A9 (VBUS), J3.B4 (VBUS), J3.B9 (VBUS)
- new net: J3.A5 (CC1), R20.1
- no-connect marks 0 -> 2
Other:
- moved on the sheet: R14, R15, R2, R3, U1F
