File: PCB/configurations.kicad_sch (KiCad schematic)
At the start: 16 parts, among them J2 Conn_ARM_SWD_TagConnect_TC2030, J3 USB_C_Receptacle_USB2.0_16P, U1 XC7A50T-FGG484, U3 FT232H

Commit message: decided on a USB to JTAG FINALLY
Parts:
- removed U3: FT232H, Package_DFN_QFN:QFN-48-1EP_8x8mm_P0.5mm_EP6.2x6.2mm_ThermalVias, symbol Interface_USB:FT232H
- added U3: FT2232HQ, Package_DFN_QFN:QFN-64-1EP_9x9mm_P0.5mm_EP4.35x4.35mm, symbol Interface_USB:FT2232HQ
Connections:
- net GND: now also U3.1 (GND), U3.10 (AGND), U3.11 (GND), U3.15 (GND), U3.25 (GND), U3.35 (GND), U3.47 (GND), U3.5 (GND), U3.51 (GND), U3.65 (GND)
